Commit message: robot moves to goal pos

File: driver_repos/ur_5e_driver/src/Universal_Robots_ROS2_Description/urdf/ur.urdf.xacro (robot description, xacro)
@@ -117,4 +117,11 @@
      <origin xyz="0 0 0" rpy="0 0 0" />          <!-- position robot in the world -->
    </xacro:ur_robot>
+   <!-- new Link for camera -->
+   <link name="$(arg tf_prefix)camera_link"/>
+    <joint name="$(arg tf_prefix)wrist_3_to_camera_joint" type="fixed">
+      <parent link="$(arg tf_prefix)wrist_3_link" />
+      <child link="$(arg tf_prefix)camera_link" />
+      <origin xyz="0.0 -0.112 0.044" rpy="0.0 0.0 -1.5708" />
+    </joint>
    <xacro:if value="$(arg sim_gazebo)">
     <!-- Gazebo plugins -->

File: driver_repos/ur_5e_driver/src/irp_ur5e_support/urdf/iras_ur5e.macro.xacro (robot description, xacro)
@@ -180,3 +180,9 @@
         <child link="tool_egh80" />
     </joint>
+    <link name="camera_link"/>
+    <joint name="wrist_3_to_camera_joint" type="fixed">
+      <parent link="wrist_3_link" />
+      <child link="camera_link" />
+      <origin xyz="0.0 -0.112 0.044" rpy="0.0 0.0 -1.5708" />
+    </joint>
 </robot>

Commit message: changed z position of camera by 2mm

File: driver_repos/ur_5e_driver/src/Universal_Robots_ROS2_Description/urdf/ur.urdf.xacro (robot description, xacro)
@@ -122,5 +122,5 @@
       <parent link="$(arg tf_prefix)wrist_3_link" />
       <child link="$(arg tf_prefix)camera_link" />
-      <origin xyz="0.0 -0.112 0.044" rpy="0.0 0.0 -1.5708" />
+      <origin xyz="0.0 -0.112 0.046" rpy="0.0 0.0 -1.5708" />
     </joint>
    <xacro:if value="$(arg sim_gazebo)">

Commit message: Wichtig, tool calibration passt für calibrator script, noch keine anpassungen für die pipeline mit tf transformationen.

File: driver_repos/ur_5e_driver/src/Universal_Robots_ROS2_Description/urdf/ur.urdf.xacro (robot description, xacro)
@@ -122,5 +122,5 @@
       <parent link="$(arg tf_prefix)wrist_3_link" />
       <child link="$(arg tf_prefix)camera_link" />
-      <origin xyz="0.0 -0.112 0.046" rpy="0.0 0.0 -1.5708" />
+      <origin xyz="-0.018 -0.112 0.07" rpy="1.5708 -1.5708 0.0" />
     </joint>
    <xacro:if value="$(arg sim_gazebo)">
